File: esp32.kicad_sch (KiCad schematic)
At the start: 25 parts, among them J1 SS-52400-002, J2 B2B-PH-SM4-TB, U1 MCP73871

Commit message: next working on that part
Parts:
- C1, C2, C5, C6: footprint (none) -> Capacitor_SMD:C_0805_2012Metric
- C3, C4: footprint (none) -> Footprints:T491A
- F1: footprint FUSC3226X100N -> Footprints:FUSC3226X100N
- J1: footprint SS-52400-002:BELFUSE_SS-52400-002 -> Footprints:BELFUSE_SS-52400-002
- J2: footprint B2B-PH-SM4-TB:JST_B2B-PH-SM4-TB -> Footprints:JST_B2B-PH-SM4-TB
- LED1, LED2, LED3, LED4: footprint LEDC2012X120N -> Footprints:LEDC2012X120N
- R1, R10, R2, R3, R4, R5, R6, R7, R8, R9: footprint (none) -> Resistor_SMD:R_0805_2012Metric
- VR1: footprint LM1117MPX-3.3:VREG_LM1117MPX-3.3 -> Footprints:VREG_LM1117MPX-3.3
Connections:
- net GND: now also U1.3 (SEL)
