File: sensors.kicad_sch (KiCad schematic)
At the start: 7 parts, among them Q1 TEMT6000X01, U6 BME280, U7 MAX4466EXK

Commit message: UI workig
Parts:
- added C15, C16, C17: 0.1u, symbol Device:C
- added R23, R25: 10K, symbol Device:R
- added R24: 100K, symbol Device:R
- added R26, R27: 1M, symbol Device:R
- added R28, R29: 2K, symbol Device:R
Connections:
- net +3.3V: now also U7.5 (VCC), C15.1, R23.1, R26.1, R28.1
- net GND: now also MK1.GND, Q1.1, U7.2 (GND), U7.3 (IN-), C15.2, C16.1, C17.1, R24.1, R25.1, R25.2, R27.2
- net PHOTO_C: now reaches Q1.3
- net PHOTO_C: now also R23.2
- net at MK1.OUT: now also U7.1 (IN+), R29.2
- net MIC_OUT: now reaches U7.4 (OUT)
- net MIC_OUT: now also C16.2, R24.2
- net SCLD renamed SCL
- net SDAD renamed SDA
- new net: R26.2, R27.1
- new net: C17.2, R28.2, R29.1
Other:
- note added: "BME 280"
- note added: "Microphone and Amplifier"
- note added: "PHOTO SENSOR"
- moved on the sheet: MK1, Q1, U7

Commit message: next working on that part
Parts:
- C14, C15, C16, C17: footprint (none) -> Capacitor_SMD:C_0805_2012Metric
- MK1: footprint CMC-5042PF-AC:CUI_CMC-5042PF-AC -> Footprints:CUI_CMC-5042PF-AC
- Q1: footprint TEMT6000X01:TRANS_TEMT6000X01 -> Footprints:TRANS_TEMT6000X01
- R21, R22, R23, R24, R25, R26, R27, R28, R29: footprint (none) -> Resistor_SMD:R_0805_2012Metric
Changed lines of the file:
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@@
 			)
 		)
-		(property "Footprint" ""
+		(property "Footprint" "Resistor_SMD:R_0805_2012Metric"
 			(at 201.422 139.7 90)
 			(effects
@@
 			)
 		)
-		(property "Footprint" ""
+		(property "Footprint" "Resistor_SMD:R_0805_2012Metric"
 			(at 240.03 151.638 90)
 			(effects
@@
 			)
 		)
-		(property "Footprint" ""
+		(property "Footprint" "Resistor_SMD:R_0805_2012Metric"
 			(at 191.262 125.73 90)
 			(effects
@@
 			)
 		)
-		(property "Footprint" "TEMT6000X01:TRANS_TEMT6000X01"
+		(property "Footprint" "Footprints:TRANS_TEMT6000X01"
 			(at 140.97 45.72 0)
 			(effects
@@
 			)
 		)
-		(property "Footprint" ""
+		(property "Footprint" "Resistor_SMD:R_0805_2012Metric"
 			(at 201.422 121.92 90)
 			(effects
@@
 			)
 		)
-		(property "Footprint" ""
+		(property "Footprint" "Capacitor_SMD:C_0805_2012Metric"
 			(at 189.23 120.9548 0)
 			(effects
@@
 			)
 		)
-		(property "Footprint" ""
+		(property "Footprint" "Capacitor_SMD:C_0805_2012Metric"
 			(at 272.7452 138.43 0)
 			(effects
@@
 			)
 		)
-		(property "Footprint" "CMC-5042PF-AC:CUI_CMC-5042PF-AC"
+		(property "Footprint" "Footprints:CUI_CMC-5042PF-AC"
 			(at 182.88 133.35 0)
 			(effects
@@
 			)
 		)
-		(property "Footprint" ""
+		(property "Footprint" "Resistor_SMD:R_0805_2012Metric"
 			(at 26.162 33.02 90)
 			(effects
@@
 			)
 		)
-		(property "Footprint" ""
+		(property "Footprint" "Resistor_SMD:R_0805_2012Metric"
 			(at 37.592 33.02 90)
 			(effects
@@
 			)
 		)
-		(property "Footprint" ""
+		(property "Footprint" "Resistor_SMD:R_0805_2012Metric"
 			(at 150.622 36.83 90)
 			(effects
@@
 			)
 		)
-		(property "Footprint" ""
+		(property "Footprint" "Resistor_SMD:R_0805_2012Metric"
 			(at 191.262 118.11 90)
 			(effects
@@
 			)
 		)
-		(property "Footprint" ""
+		(property "Footprint" "Capacitor_SMD:C_0805_2012Metric"
 			(at 91.1352 45.72 0)
 			(effects
@@
 			)
 		)
-		(property "Footprint" ""
+		(property "Footprint" "Capacitor_SMD:C_0805_2012Metric"
 			(at 243.84 155.2448 0)
 			(effects
@@
 			)
 		)
-		(property "Footprint" ""
+		(property "Footprint" "Resistor_SMD:R_0805_2012Metric"
 			(at 207.772 142.24 90)
 			(effects
