File: user_interface.kicad_sch (KiCad schematic)
At the start: 0 parts

Commit message: UI workig
Parts:
- added J4: Conn_01x04_Pin, symbol Connector:Conn_01x04_Pin
Changed lines of the file:
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@@
 	(generator_version "9.0")
 	(paper "A4")
+	(symbol
+		(lib_id "Connector:Conn_01x04_Pin")
+		(at 46.99 31.75 0)
+		(unit 1)
+		(exclude_from_sim no)
+		(in_bom yes)
+		(on_board yes)
+		(dnp no)
+		(fields_autoplaced yes)
+		(property "Reference" "J4"
+			(at 47.625 24.13 0)
+			(effects
+				(font
+					(size 1.27 1.27)
+				)
+			)
+		)
+		(property "Value" "Conn_01x04_Pin"
+			(at 47.625 26.67 0)
+			(effects
+				(font
+					(size 1.27 1.27)
+				)
+			)
+		)
+		(property "Footprint" ""
+			(at 46.99 31.75 0)
+			(effects
+				(font
+					(size 1.27 1.27)
+				)
+				(hide yes)
+			)
+		)
+		(property "Datasheet" "~"
+			(at 46.99 31.75 0)
+			(effects
+				(font
+					(size 1.27 1.27)
+				)
+				(hide yes)
+			)
+		)
+		(property "Description" "Generic connector, single row, 01x04, script generated"
+			(at 46.99 31.75 0)
+			(effects
+				(font
+					(size 1.27 1.27)
+				)
+				(hide yes)
+			)
+		)
+		(pin "2"
+		)
+		(pin "1"
+		)
+		(pin "3"
+		)
+		(pin "4"
+		)
+		(instances
+			(project ""
+				(path "/3a4906cd-b970-47fd-b3df-3da3a46542f3/ce9639a1-645c-4d9b-b86e-887c0addc46e/b2d67d36-6f28-4ae0-9f74-73bfed45a312"
+					(reference "J4")
+					(unit 1)
+				)
+			)
+		)
+	)
 )

Commit message: latest new dev
Parts:
- added C18: 0.1u, symbol Device:C
- added C19: 1u, symbol Device:C
- added J5: Conn_01x05_Pin, symbol Connector:Conn_01x05_Pin
- added Q2, Q3: BC817, Package_TO_SOT_SMD:SOT-23, symbol Transistor_BJT:BC817
- added R30, R31, R32: 10K, symbol Device:R
- added S1: Boot, USLPT2819DT2TR:SW_USLPT2819DT2TR, symbol USLPT2819DT2TR:USLPT2819DT2TR
- added S2: USLPT2819DT2TR, USLPT2819DT2TR:SW_USLPT2819DT2TR, symbol USLPT2819DT2TR:USLPT2819DT2TR
Connections:
- net GND: now reaches J4.1 (Pin_1)
- net GND: now also C18.2, C19.2, J5.1 (Pin_1), S1.1, S1.2, S2.1, S2.2
- net SCL: now reaches J4.2 (Pin_2)
- net SDA: now reaches J4.3 (Pin_3)
- net +3.3V: now reaches J4.4 (Pin_4)
- net +3.3V: now also J5.5 (Pin_5), R32.1
- new net: Q3.1 (B), R31.2
- new net: Q2.1 (B), R30.2
- new net BOOT: C18.1, Q3.2 (E), S1.3, S1.4
- new net DTR: Q3.3 (C), R30.1
- new net EN: C19.1, Q2.3 (C), R32.2, S2.3, S2.4
- new net GPIO18: J5.3 (Pin_3)
- new net GPIO8: J5.4 (Pin_4)
- new net GPIO819: J5.2 (Pin_2)
- new net RTS: Q2.2 (E), R31.1
Other:
- note added: "Breakout for Remaining Pins"
- note added: "ESP32 Boot mode"
- note added: "OLED display connectors (12C)"
- note added: "Reset and Boot button"
- moved on the sheet: J4

Commit message: next working on that part
Parts:
- C18, C19: footprint (none) -> Capacitor_SMD:C_0805_2012Metric
- J4: footprint (none) -> Connector_PinHeader_2.54mm:PinHeader_1x04_P2.54mm_Vertical
- J5: footprint (none) -> Connector_PinHeader_2.54mm:PinHeader_1x05_P2.54mm_Vertical
- R30, R31, R32: footprint (none) -> Resistor_SMD:R_0805_2012Metric
- S1, S2: footprint USLPT2819DT2TR:SW_USLPT2819DT2TR -> Footprints:SW_USLPT2819DT2TR
Changed lines of the file:
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@@
 			)
 		)
-		(property "Footprint" ""
+		(property "Footprint" "Connector_PinHeader_2.54mm:PinHeader_1x04_P2.54mm_Vertical"
 			(at 55.88 39.37 0)
 			(effects
@@
 			)
 		)
-		(property "Footprint" ""
+		(property "Footprint" "Connector_PinHeader_2.54mm:PinHeader_1x05_P2.54mm_Vertical"
 			(at 58.42 74.93 0)
 			(effects
@@
 			)
 		)
-		(property "Footprint" ""
+		(property "Footprint" "Resistor_SMD:R_0805_2012Metric"
 			(at 111.76 93.218 90)
 			(effects
@@
 			)
 		)
-		(property "Footprint" ""
+		(property "Footprint" "Capacitor_SMD:C_0805_2012Metric"
 			(at 98.7552 49.53 0)
 			(effects
@@
 			)
 		)
-		(property "Footprint" "USLPT2819DT2TR:SW_USLPT2819DT2TR"
+		(property "Footprint" "Footprints:SW_USLPT2819DT2TR"
 			(at 110.49 33.02 0)
 			(effects
@@
 			)
 		)
-		(property "Footprint" ""
+		(property "Footprint" "Resistor_SMD:R_0805_2012Metric"
 			(at 111.76 77.978 90)
 			(effects
@@
 			)
 		)
-		(property "Footprint" ""
+		(property "Footprint" "Capacitor_SMD:C_0805_2012Metric"
 			(at 140.6652 53.34 0)
 			(effects
@@
 			)
 		)
-		(property "Footprint" "USLPT2819DT2TR:SW_USLPT2819DT2TR"
+		(property "Footprint" "Footprints:SW_USLPT2819DT2TR"
 			(at 148.59 38.1 0)
 			(effects
@@
 			)
 		)
-		(property "Footprint" ""
+		(property "Footprint" "Resistor_SMD:R_0805_2012Metric"
 			(at 134.112 33.02 90)
 			(effects
